File: MouseKeyboard.sch (KiCad schematic (older format))
At the start: 16 parts, among them J1 USB, SW1 SPST, SW2 SW_PUSH, SW3 SW_PUSH, SW4 SW_PUSH, SW5 SW_PUSH, SW6 SW_PUSH, SW7 SW_PUSH, SW8 SW_PUSH, U1 2AxisPotWSelect

Commit message: Changed Paper Size
Parts:
- removed D1, D2: DIODESCH, symbol DIODESCH
- removed J1: USB, symbol USB
- removed R1: 2K2, symbol R
- removed R2, R3: 68R, symbol R
- removed SHIELD1: ARDUINO_SHIELD, symbol ARDUINO_SHIELD
- removed SW1: SPST, symbol SPST
- removed SW2, SW3, SW4, SW5, SW6, SW7, SW8: SW_PUSH, symbol SW_PUSH
- removed U1: 2AxisPotWSelect, symbol 2AxisPotWSelect
- added D? (x2): DIODESCH, symbol DIODESCH
- added IC?: ATMEGA328P-P, DIL28, symbol ATMEGA328P-P
- added J?: USB, symbol USB
- added R? (x2): 68R, symbol R
- added R?: 2K2, symbol R
- added U?: 2AxisPotWSelect, symbol 2AxisPotWSelect
Connections:
- net labels added: +5V, GND, XTAL1, XTAL2
- wire segments 76 -> 40
- no-connect marks 13 -> 4
Other:
- note added: "Pin2\n"
- note added: "Pin7\n"

Commit message: Schematic is almost complete!!!
The schematic just needs to be annotated, and values added. Then it
is done.
Parts:
- added C1, C2: C, symbol C
- added R4: 1M, symbol R
- added SW1, SW2, SW3, SW4, SW5, SW6, SW7: SW_PUSH, symbol SW_PUSH
- added SW8: SPST, symbol SPST
- added X1: CRYSTAL, symbol CRYSTAL
- gave numbers to parts that had none: 8
Connections:
- net +5V: now also SW1.2, SW2.2, SW3.2, SW4.2, SW5.2, SW6.2, SW7.2, SW8.1
- net GND: now also C1.2, C2.2
- net XTAL1: now also C1.1, R4.1, X1.1
- net XTAL2: now also C2.1, R4.2, X1.2
- net at IC1.11 ((PCINT21/OC0B/T1)PD5): now also SW2.1
- net at IC1.12 ((PCINT22/OC0A/AIN0)PD6): now also SW3.1
- net at IC1.14 ((PCINT0/CLKO/ICP1)PB0): now also SW4.1
- net at IC1.15 ((PCINT1/OC1A)PB1): now also SW5.1
- net at IC1.16 ((PCINT2/OC1B/~SS~)PB2): now also SW6.1
- net at IC1.17 ((PCINT3/OC2A/MOSI)PB3): now also SW7.1
- net at IC1.18 ((PCINT4/MISO)PB4): now also SW8.2
- net at IC1.6 ((PCINT20/XCK/T0)PD4): now also SW1.1
- no-connect marks 4 -> 11

Commit message: Finished The Pcb Parts List
Parts:
- C1, C2: value C -> 22P
- X1: value CRYSTAL -> CRYSTAL-16MHz
Connections:
- no-connect marks 11 -> 12
Changed lines of the file:
@@
 P 11450 6150
 F 0 "X1" H 11450 6300 60  0000 C CNN
-F 1 "CRYSTAL" H 11450 6000 60  0000 C CNN
+F 1 "CRYSTAL-16MHz" H 11450 6000 60  0000 C CNN
 F 2 "" H 11450 6150 60  0000 C CNN
 F 3 "" H 11450 6150 60  0000 C CNN
@@
 P 12000 5950
 F 0 "C1" H 12000 6050 40  0000 L CNN
-F 1 "C" H 12006 5865 40  0000 L CNN
+F 1 "22P" H 12006 5865 40  0000 L CNN
 F 2 "" H 12038 5800 30  0000 C CNN
 F 3 "" H 12000 5950 60  0000 C CNN
@@
 P 12000 6350
 F 0 "C2" H 12000 6450 40  0000 L CNN
-F 1 "C" H 12006 6265 40  0000 L CNN
+F 1 "22P" H 12006 6265 40  0000 L CNN
 F 2 "" H 12038 6200 30  0000 C CNN
 F 3 "" H 12000 6350 60  0000 C CNN
@@
 NoConn ~ 4200 5150
 NoConn ~ 4200 4300
+NoConn ~ 2700 500
 $EndSCHEMATC

Commit message: Just a commit
Restarted Laying out pcb
Changed lines of the file:
@@
 LIBS:2axispotwselect
 LIBS:MouseKeyboard-cache
-LIBS:Sheet2-cache
 EELAYER 24 0
 EELAYER END
@@
 Wire Wire Line
 	5150 6600 5150 6350
-Connection ~ 2050 6100
 Connection ~ 2050 6000
 Wire Wire Line
 	2050 6000 2050 6650
-Wire Wire Line
-	2300 6100 2050 6100
-Wire Wire Line
-	5050 4750 4200 4750
-Wire Wire Line
-	5050 6600 5050 4750
-Wire Wire Line
-	4950 4650 4950 6600
-Wire Wire Line
-	4200 4650 4950 4650
 Wire Wire Line
 	4850 5700 4850 6600
@@
 NoConn ~ 4200 4300
 NoConn ~ 2700 500
+$Comp
+L GND #PWR?
+U 1 1 54DEC1FA
+P 2200 6650
+F 0 "#PWR?" H 2200 6650 30  0001 C CNN
+F 1 "GND" H 2200 6580 30  0001 C CNN
+F 2 "" H 2200 6650 60  0000 C CNN
+F 3 "" H 2200 6650 60  0000 C CNN
+	1    2200 6650
+	1    0    0    -1
+$EndComp
+Wire Wire Line
+	2300 6100 2200 6100
+Wire Wire Line
+	2200 6100 2200 6650
+Wire Wire Line
+	5050 6600 5050 4750
+Wire Wire Line
+	5050 4750 4200 4750
+Wire Wire Line
+	4200 4650 4950 4650
+Wire Wire Line
+	4950 4650 4950 6600
 $EndSCHEMATC
